File: kicad/raw_hall_elements/raw_hall_elements.kicad_sch (KiCad schematic)
At the start: 23 parts, among them J1 Conn_01x03_Socket, J2 Conn_01x02_Socket, U1 MCP6022

Commit message: Schematic now uses smaller opamp
Parts:
- removed R14, R15: 200, Resistor_SMD:R_0603_1608Metric, symbol Device:R
- removed U1: MCP6022, Package_SO:SOIC-8-N7_3.9x4.9mm_P1.27mm, symbol Amplifier_Operational:MCP6022
- added U1: LMV358, Package_DFN_QFN:OnSemi_UDFN-8_1.2x1.8mm_P0.4mm, symbol Amplifier_Operational:LMV358
Connections:
- net +3V3: now also U1.8 (V+)
- net GND: now also U1.4 (V-)
- net Hall1_out+: now also R13.1
- net Hall2_out+: now also R16.1
- net Vout1: now also U1.1
- net Vout2: now also U1.7
- net at R5.1: now also U1.6 (-)
- net at R2.2, R3.1: now also U1.5 (+)
- net at R1.2, R4.1: now also U1.3 (+)
- net at R6.1: now also U1.2 (-)

Commit message: more progress
Parts:
- removed HALL_ELEMENT_1_IN1, HALL_ELEMENT_2_IN1: Conn_01x04, Connector_PinSocket_2.00mm:PinSocket_1x04_P2.00mm_Horizontal, symbol Connector_Generic:Conn_01x04
- removed J1: Conn_01x03_Socket, Connector_JST:JST_EH_S2B-EH_1x02_P2.50mm_Horizontal, symbol Connector:Conn_01x03_Socket
- removed J2: Conn_01x02_Socket, Connector_JST:JST_EH_S2B-EH_1x02_P2.50mm_Horizontal, symbol Connector:Conn_01x02_Socket
- removed R12, R18: 1.5k, Resistor_SMD:R_0603_1608Metric, symbol Device:R
- added 3V3, 5V1, GND1, VO1, VO2: Conn_01x01, TestPoint:TestPoint_THTPad_1.0x1.0mm_Drill0.5mm, symbol Connector_Generic:Conn_01x01
- added IC1, IC2: AHE300G-PA4-B, KiCad:AHE300GPA4B, symbol AHE300G-PA4-B:AHE300G-PA4-B
Connections:
- net +3V3: now also 3V3.1 (Pin_1)
- net +5V: now also 5V1.1 (Pin_1)
- net GND: now also R11.2, R17.2, GND1.1 (Pin_1), IC1.3 (INPUT(-+)), IC1.4 (OUTPUT(-+)), IC2.3 (INPUT(-+)), IC2.4 (OUTPUT(-+))
- net Hall1_out+: now also IC1.2 (OUTPUT(+-))
- net Hall2_out+: now also IC2.2 (OUTPUT(+-))
- net Vin+: now also IC1.1 (INPUT(+-)), IC2.1 (INPUT(+-))
- net Vout1: now also VO1.1 (Pin_1)
- net Vout2: now also VO2.1 (Pin_1)

Commit message: one more trace ahhhhh
Parts:
- removed U1: LMV358, Package_DFN_QFN:OnSemi_UDFN-8_1.2x1.8mm_P0.4mm, symbol Amplifier_Operational:LMV358
- added U2: MCP6002-xMS, Package_SO:MSOP-8_3x3mm_P0.65mm, symbol Amplifier_Operational:MCP6002-xMS
Connections:
- net +3V3: now also U2.8 (V+)
- net GND: now also U2.4 (V-)
- net Vout1: now also U2.1
- net Vout2: now also U2.7
- net at R5.1: now also U2.6 (-)
- net at R2.2, R3.1: now also U2.5 (+)
- net at R1.2, R4.1: now also U2.3 (+)
- net at R6.1: now also U2.2 (-)

Commit message: schematic clean up and layout finalise
Parts:
- 3V3, 5V1, GND1, VO1, VO2: footprint TestPoint:TestPoint_THTPad_1.0x1.0mm_Drill0.5mm -> TestPoint:TestPoint_THTPad_1.5x1.5mm_Drill0.7mm
Other:
- moved on the sheet: 3V3, 5V1, GND1, IC1, IC2, R1, R10, R11, R13, R16, R17, R2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
